Commit message: envs

File: data/robots/ur5/ur5_robotiq85_on_table.urdf (robot description, URDF)
Before this commit: robot ur5, 10 links, 9 joints
Links:
- removed link base
- added link table; collision box size=0.7 2.0 0.01; visual box size=0.7 2.0 0.01
- link tool: geometry collision cylinder length=0.1 radius=0.01; visual cylinder length=0.1 radius=0.01
Joints:
- removed joint base_link-base_fixed_joint
- added joint table_joint: type fixed, parent table, child base_link, origin xyz=0.0 0.0 0.0 rpy=0.0 0.0 0.0
